Commit message: removed comment

File: simple_grace.urdf (robot description, URDF)
Before this commit: robot grace, 17 links, 16 joints
Links:
- link LF-FOOT: geometry visual sphere radius=0.02
- link LF-KFE: geometry collision cylinder length=0.13 radius=0.015; visual cylinder length=0.3 radius=0.015
- link LR-FOOT: geometry visual sphere radius=0.02
- link LR-KFE: geometry collision cylinder length=0.13 radius=0.015; visual cylinder length=0.3 radius=0.015
- link RF-FOOT: geometry visual sphere radius=0.02
- link RF-KFE: geometry collision cylinder length=0.13 radius=0.015; visual cylinder length=0.3 radius=0.015
- link RR-KFE: geometry collision cylinder length=0.13 radius=0.015; visual cylinder length=0.3 radius=0.015
- link grace: mass 10 -> 1.0
Joints:
- joint LF-KFE_LF-FOOT: origin xyz=0 0.17 0 rpy=0 0 0 -> xyz=0 0.31 0 rpy=0 0 0
- joint LR-KFE_LR-FOOT: origin xyz=0 0.17 0 rpy=0 0 0 -> xyz=0 0.31 0 rpy=0 0 0
- joint RF-KFE_RF-FOOT: origin xyz=0 0.17 0 rpy=0 0 0 -> xyz=0 0.31 0 rpy=0 0 0
- joint RR-KFE_RR-FOOT: origin xyz=0 0.17 0 rpy=0 0 0 -> xyz=0 0.31 0 rpy=0 0 0
